File: Electronics/Mainboard.brd (EAGLE design)
At the start: 68.6 x 53.3 mm, 10 parts, among them IC1 ER400RTS-02

Commit message: Changed pin 5 and 9. Closes #42
Connections:
- net N$16: now also U$1.D5; no longer U$1.D9
- net N$8: now also U$1.D9; no longer U$1.D5
Routing:
- net N$8: track 18.0 -> 15.3 mm
- net N$16: track 15.5 -> 13.4 mm
